File: board/schem/schem.kicad_pcb (KiCad board)
At the start: 2 copper layers, 133 x 87 mm, 160 parts, among them J1 no_break, J10 no_hal, J11 break2, J12 impulse, J13 hal, J14 no_temp, J15 speed, J16 analog, J18 adc_red1, J19 adc_red2, J2 motor_out, J20 ON/OFF, J21 lamp, J3 test, J4 motor_tmp, J8 POWER_IN, J9 break1, Q1 BC817, Q10 BC817, Q11 BC817, Q12 BC817, Q2 BC817, Q3 BC817, Q4 BC817, Q5 BC817, Q6 BC817, Q7 BC817, Q8 BC817, Q9 BC817, SW1 SW_Push, SW2 SW_Push, T1 NTD5865NL, T2 FDD9507L, T3 NTD5865NL, T4 FDD9507L, T5 NTD5865NL, T6 FDD9507L, U1 CFPS-39-12M, U10 AP2138, U11 LD1117, U12 68u, U2 EP4CE6, U3 JTAG, U4 IS25LQ, U5 LF33CDT, U6 IS25LQ, U7 MPC3008, U8 A8498, U9 B350B

Commit message: some  tests
Parts:
- removed J16: analog, Connector_PinSocket_2.54mm:PinSocket_1x02_P2.54mm_Vertical
- removed J19: adc_red2, Connector_PinSocket_2.54mm:PinSocket_1x03_P2.54mm_Vertical
- added J5: motor_tmp, Connector_PinSocket_2.54mm:PinSocket_1x02_P2.54mm_Vertical, F.Cu at (245.8, -13.0)
- added J6: adc_red1, Connector_PinSocket_2.54mm:PinSocket_1x03_P2.54mm_Vertical, F.Cu at (241.2, -13.0)
- added Q13: BC817, Package_TO_SOT_SMD:SOT-23, F.Cu at (210.9, 8.43)
- added R69: 10k, Resistor_SMD:R_1206_3216Metric, F.Cu at (250.9, -13.7)
- added R70: 10k, Resistor_SMD:R_1206_3216Metric, F.Cu at (246.3, -6.50)
- added R71: 10k, Resistor_SMD:R_1206_3216Metric, F.Cu at (250.9, -10.4)
- added R72: 10k, Resistor_SMD:R_1206_3216Metric, F.Cu at (256.5, -13.7)
- added R73: 4.7k, Resistor_SMD:R_1206_3216Metric, F.Cu at (251.9, -7.07)
- added R74: 50k, Resistor_SMD:R_1206_3216Metric, F.Cu at (205.9, 7.80)
- D14: value 3.3V_led -> 2.5V_led
- D15: value 3.3V_led -> 1.2V_led
- R20: value 8k -> 2.4
- R35, R62, R64: value 10k -> 90k
- R49, R63, R65: value 10k -> 5k
- R5, R53, R7: value 3k -> 1k
- R58, R8: value 8k -> 2.4k
- T1: value NTD5865NL -> CDZ44-CDI; footprint Package_TO_SOT_SMD:TO-252-2 -> Package_TO_SOT_THT:TO-220-3_Vertical; moved to F.Cu
- T2: value FDD9507L -> IRF4905; footprint Package_TO_SOT_SMD:TO-252-2 -> Package_TO_SOT_THT:TO-220-3_Vertical; moved to F.Cu
- T3, T5: value NTD5865NL -> CDZ44-CDI; footprint Package_TO_SOT_SMD:TO-252-2 -> Package_TO_SOT_THT:TO-220-3_Vertical
- T4, T6: value FDD9507L -> IRF4905; footprint Package_TO_SOT_SMD:TO-252-2 -> Package_TO_SOT_THT:TO-220-3_Vertical
- moved T1 152.9 mm to (206.3, -11.4)
- moved T2 143.2 mm to (206.3, -5.41)
- moved D3 78.1 mm to (76.3, 12.8)
- moved T3 74.3 mm to (217.8, -11.4)
- moved T5 60.8 mm to (217.8, -5.41)
- moved T6 32.9 mm to (217.8, 0.55)
- moved T4 22.5 mm to (206.3, 0.55)
Connections:
- C11 pad 1: +36V -> Net-(C11-Pad1)
- C18 pad 1: +36V -> Net-(C11-Pad1)
- D15 pad 1: GND -> Net-(D15-Pad1)
- F1 pad 1: Net-(F1-Pad1) -> +36V
- J13 pad 2: Net-(J13-Pad2) -> (no net)
- J15 pad 2: +5V -> +3V3
- J18 pad 2: +5V -> +3V3
- J18 pad 3: /control/red1 -> /control/spare_2
- J20 pad 1: Net-(F1-Pad1) -> Net-(C11-Pad1)
- R48 pad 2: +1V2 -> +3V3
- R67 pad 2: +5V -> +3V3
- T2 pad 2: /DriveAndSens/A_out -> +36V
- T2 pad 3: +36V -> /DriveAndSens/A_out
- T4 pad 2: /DriveAndSens/B_out -> +36V
- T4 pad 3: +36V -> /DriveAndSens/B_out
- T6 pad 2: /DriveAndSens/C_out -> +36V
- T6 pad 3: +36V -> /DriveAndSens/C_out
- U1 pad 1: Net-(U1-Pad1) -> (no net)
- U2 pad 1: Net-(U2-Pad1) -> (no net)
- U2 pad 10: Net-(U2-Pad10) -> (no net)
- U2 pad 100: Net-(U2-Pad100) -> (no net)
- U2 pad 101: Net-(U2-Pad101) -> (no net)
- U2 pad 11: Net-(U2-Pad11) -> (no net)
- U2 pad 119: Net-(U2-Pad119) -> (no net)
- U2 pad 120: Net-(U2-Pad120) -> (no net)
- U2 pad 121: Net-(U2-Pad121) -> (no net)
- U2 pad 124: Net-(U2-Pad124) -> (no net)
- U2 pad 125: Net-(U2-Pad125) -> (no net)
- U2 pad 126: Net-(U2-Pad126) -> (no net)
- U2 pad 127: Net-(U2-Pad127) -> (no net)
- U2 pad 135: Net-(U2-Pad135) -> (no net)
- U2 pad 136: Net-(U2-Pad136) -> (no net)
- U2 pad 137: Net-(U2-Pad137) -> (no net)
- U2 pad 138: Net-(U2-Pad138) -> (no net)
- U2 pad 141: Net-(U2-Pad141) -> (no net)
- U2 pad 142: Net-(U2-Pad142) -> (no net)
- U2 pad 143: Net-(U2-Pad143) -> (no net)
- U2 pad 144: Net-(U2-Pad144) -> (no net)
- U2 pad 2: Net-(U2-Pad2) -> (no net)
- U2 pad 25: Net-(U2-Pad25) -> (no net)
- U2 pad 28: Net-(U2-Pad28) -> (no net)
- U2 pad 3: Net-(U2-Pad3) -> (no net)
- U2 pad 42: Net-(U2-Pad42) -> (no net)
- U2 pad 46: Net-(U2-Pad46) -> (no net)
- U2 pad 49: Net-(U2-Pad49) -> (no net)
- U2 pad 52: Net-(U2-Pad52) -> (no net)
- U2 pad 53: Net-(U2-Pad53) -> (no net)
- U2 pad 54: Net-(U2-Pad54) -> (no net)
- U2 pad 55: Net-(U2-Pad55) -> (no net)
- U2 pad 58: Net-(U2-Pad58) -> (no net)
- U2 pad 59: Net-(U2-Pad59) -> (no net)
- U2 pad 60: Net-(U2-Pad60) -> (no net)
- U2 pad 64: Net-(U2-Pad64) -> (no net)
- U2 pad 65: Net-(U2-Pad65) -> (no net)
- U2 pad 66: Net-(U2-Pad66) -> (no net)
- U2 pad 7: Net-(U2-Pad7) -> (no net)
- U2 pad 73: Net-(U2-Pad73) -> (no net)
- U2 pad 74: Net-(U2-Pad74) -> (no net)
- U2 pad 75: Net-(U2-Pad75) -> (no net)
- U2 pad 76: Net-(U2-Pad76) -> (no net)
- U2 pad 77: Net-(U2-Pad77) -> (no net)
- U2 pad 80: Net-(U2-Pad80) -> (no net)
- U2 pad 83: Net-(U2-Pad83) -> (no net)
- U2 pad 84: Net-(U2-Pad84) -> (no net)
- U2 pad 85: Net-(U2-Pad85) -> (no net)
- U2 pad 86: Net-(U2-Pad86) -> (no net)
- U2 pad 87: Net-(U2-Pad87) -> (no net)
- U2 pad 88: Net-(U2-Pad88) -> (no net)
- U2 pad 89: Net-(U2-Pad89) -> (no net)
- U2 pad 90: Net-(U2-Pad90) -> (no net)
- U2 pad 91: Net-(U2-Pad91) -> (no net)
- U2 pad 99: Net-(U2-Pad99) -> (no net)
- U3 pad 6: Net-(U3-Pad6) -> (no net)
- U3 pad 7: Net-(U3-Pad7) -> (no net)
- U3 pad 8: Net-(U3-Pad8) -> (no net)
- U7 pad 3: /control/red1 -> /control/temp_tran
- U7 pad 4: /control/red2 -> /control/spare_1
- U7 pad 5: /control/ch1 -> /control/spare_2
- U8 pad 8: +36V -> Net-(C11-Pad1)
Routing:
- net GND: track 909.0 -> 0.00 mm, vias 23 -> 0
- net +3V3: track 705.6 -> 0.00 mm, vias 18 -> 0
- net +36V: track 337.2 -> 0.00 mm, vias 6 -> 0
- net +1V2: track 245.8 -> 0.00 mm, vias 6 -> 0
- net +2V5: track 208.5 -> 0.00 mm, vias 6 -> 0
- net /DriveAndSens/A_n: track 201.1 -> 0.00 mm, vias 1 -> 0
- net /DriveAndSens/A_p: track 187.0 -> 0.00 mm, vias 1 -> 0
- net +5V: track 170.1 -> 0.00 mm, vias 5 -> 0
- net /DriveAndSens/B_p: track 100.0 -> 0.00 mm, vias 1 -> 0
- net /DriveAndSens/B_n: track 99.5 -> 0.00 mm, vias 1 -> 0
- net /DriveAndSens/A_out: track 94.0 -> 0.00 mm, vias 1 -> 0
- net /DriveAndSens/B_out: track 80.1 -> 0.00 mm
- net /DriveAndSens/C_out: track 70.9 -> 0.00 mm
- net /control/hal_C: track 70.5 -> 0.00 mm, vias 1 -> 0
- net /control/D_hal: track 68.2 -> 0.00 mm
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- removed copper zone on B.Cu, net GND
- removed copper zone on F.Cu, net GND
Other:
- board size 133 x 87 mm -> 133 x 67 mm

Commit message: work on  schema
Parts:
- removed R27, R3, R6: 400k, Resistor_SMD:R_1206_3216Metric
- C24: moved to F.Cu
- D10, D12, D13, D14, D15, D3, D4, D9, Q10, Q13, Q2, Q4, Q5, Q6, Q7, Q8, R20, R45, R46, R47, R48, R5, R53, R58, R74: moved to B.Cu
- R1, R2, R26: value 2k -> 50k; moved to B.Cu
- R10: value 4k -> 2k
- R21, R22, R59: value 100k -> 20k; moved to B.Cu
- R23: value 100k -> 50k
- R24, R60: value 10k -> 5k; moved to B.Cu
- R25, R61: value 4k -> 2k; moved to B.Cu
- R34, R4: value 100k -> 50k; moved to B.Cu
- R9: value 10k -> 5k
- moved R72 186.9 mm to (105.6, 96.8), turned to 270 degrees
- moved R71 173.9 mm to (105.4, 85.0), turned to 270 degrees
- moved R69 173.4 mm to (108.3, 85.0), turned to 270 degrees
- moved R70 172.2 mm to (108.5, 96.8), turned to 90 degrees
- moved J2 151.3 mm to (7.70, 88.7)
- moved R66 138.0 mm to (115.4, 83.1), turned to 180 degrees
- moved Q1 135.1 mm to (194.3, 18.3), turned to 90 degrees
- moved J20 133.9 mm to (220.0, 132.8), turned to 0 degrees
- moved R52 133.3 mm to (108.1, 122.1), turned to 180 degrees
- moved R10 131.5 mm to (184.4, 12.2), turned to 0 degrees
- moved R54 131.2 mm to (108.1, 119.4), turned to 0 degrees
- moved R8 129.4 mm to (193.0, 14.1), turned to 270 degrees
- moved R23 128.9 mm to (189.5, 21.4), turned to 180 degrees
- moved R9 127.6 mm to (189.4, 16.2)
- moved J8 127.2 mm to (224.9, 121.7), turned to 180 degrees
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Routing:
- net (no net): vias 0 -> 1
Other:
- board size 133 x 67 mm -> 133 x 77 mm
