File: board/schem/schem.kicad_pcb (KiCad board)
At the start: 2 copper layers, 133 x 77 mm, 164 parts, among them J1 no_break, J10 no_hal, J11 break2, J12 impulse, J13 hal, J14 no_temp, J15 speed, J18 adc_red1, J2 motor_out, J20 ON/OFF, J21 lamp, J3 test, J4 motor_tmp, J5 motor_tmp, J6 adc_red1, J8 POWER_IN, J9 break1, Q1 BC817, Q10 BC817, Q11 BC817, Q12 BC817, Q13 BC817, Q2 BC817, Q3 BC817, Q4 BC817, Q5 BC817, Q6 BC817, Q7 BC817, Q8 BC817, Q9 BC817, SW1 SW_Push, SW2 SW_Push, T1 CDZ44-CDI, T2 IRF4905, T3 CDZ44-CDI, T4 IRF4905, T5 CDZ44-CDI, T6 IRF4905, U1 CFPS-39-12M, U10 AP2138, U11 LD1117, U12 68u, U2 EP4CE6, U3 JTAG, U4 IS25LQ, U5 LF33CDT, U6 IS25LQ, U7 MPC3008, U8 A8498, U9 B350B

Commit message: work  on schema
Parts:
- moved R68 138.9 mm to (204.7, 109.1), turned to 90 degrees
- moved J2 105.8 mm to (113.1, 80.2)
- moved J21 88.2 mm to (197.0, 126.5)
- moved R8 71.4 mm to (217.9, 81.1), turned to 180 degrees
- moved Q1 70.4 mm to (217.7, 84.7)
- moved D12 70.3 mm to (153.9, 96.6)
- moved D13 70.3 mm to (140.0, 88.6)
- moved D2 70.3 mm to (198.7, 88.1)
- moved D3 70.3 mm to (183.0, 96.1)
- moved Q10 70.3 mm to (149.0, 84.0)
- moved Q2 70.3 mm to (189.7, 84.3)
- moved Q3 70.3 mm to (207.1, 82.5)
- moved Q4 70.3 mm to (207.2, 86.9)
- moved Q6 70.3 mm to (179.6, 83.2)
- moved Q8 70.3 mm to (149.1, 88.4)
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Routing:
- net GND: track 0.00 -> 42.6 mm, vias 0 -> 4
- net +1V2: track 0.00 -> 14.7 mm, vias 0 -> 2
- net +2V5: track 0.00 -> 11.5 mm, vias 0 -> 2
- net +3V3: track 0.00 -> 7.35 mm, vias 0 -> 1
Other:
- board size 133 x 77 mm -> 129.8 x 66 mm
- net class energy: trace_width 3.5 -> 2.5
- net class energy_mid: trace_width 3 -> 2.5; via_dia 0.8 -> 4

Commit message: work on schema
Parts:
- moved J14 80.6 mm to (119.3, 75.4), turned to 0 degrees
- moved J10 71.5 mm to (125.9, 75.4), turned to 0 degrees
- moved R33 69.5 mm to (124.0, 82.0), turned to 90 degrees
- moved J2 67.8 mm to (175.2, 107.5), turned to 180 degrees
- moved J1 64.6 mm to (133.0, 75.3), turned to 0 degrees
- moved R30 61.1 mm to (128.1, 82.0), turned to 90 degrees
- moved R28 53.8 mm to (132.6, 82.0), turned to 90 degrees
- moved R38 43.3 mm to (128.2, 130.5), turned to 0 degrees
- moved SW2 37.6 mm to (127.9, 126.1), turned to 90 degrees
- moved R5 26.1 mm to (192.0, 104.8)
- moved R2 26.1 mm to (197.2, 113.0)
- moved R22 26.1 mm to (192.2, 110.3)
- moved Q2 26.1 mm to (197.2, 109.3)
- moved R4 26.1 mm to (192.1, 113.0)
- moved R25 26.1 mm to (186.8, 104.4)
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Connections:
- U2 pad 1: (no net) -> /control/SI_1
- U2 pad 113: /control/n_b -> (no net)
- U2 pad 114: /control/n_h -> (no net)
- U2 pad 115: /control/n_t -> (no net)
- U2 pad 128: /control/SO_1 -> (no net)
- U2 pad 129: /control/SCK_1 -> (no net)
- U2 pad 132: /control/nCE_1 -> (no net)
- U2 pad 133: /control/SI_1 -> (no net)
- U2 pad 143: (no net) -> /control/SO_1
- U2 pad 144: (no net) -> /control/SCK_1
- U2 pad 2: (no net) -> /control/nCE_1
- U2 pad 89: (no net) -> /control/n_b
- U2 pad 90: (no net) -> /control/n_h
- U2 pad 91: (no net) -> /control/n_t
- U7 pad 15: +5V -> +3V3
Routing:
- net GND: track 42.6 -> 487.6 mm, vias 4 -> 11
- net +3V3: track 7.35 -> 434.8 mm, vias 1 -> 6
- net +36V: track 0.00 -> 201.2 mm, vias 0 -> 1
- net +1V2: track 14.7 -> 118.9 mm, vias 2 -> 8
- net /DriveAndSens/A_p: track 0.00 -> 83.0 mm, vias 0 -> 3
- net /DriveAndSens/A_n: track 0.00 -> 78.6 mm, vias 0 -> 3
- net +5V: track 0.00 -> 70.7 mm, vias 0 -> 2
- net /DriveAndSens/C_out: track 0.00 -> 68.9 mm
- net /DriveAndSens/B_n: track 0.00 -> 63.6 mm, vias 0 -> 3
- net Net-(Q3-Pad3): track 0.00 -> 62.6 mm, vias 0 -> 1
- net /DriveAndSens/A_out: track 0.00 -> 61.0 mm
- net Net-(C11-Pad1): track 0.00 -> 60.9 mm, vias 0 -> 1
- net Net-(C17-Pad1): track 0.00 -> 56.0 mm, vias 0 -> 1
- net /control/spare_2: track 0.00 -> 54.3 mm, vias 0 -> 1
- net /control/nCEO: track 0.00 -> 46.3 mm
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
Commit message: working on  schema
Parts:
- moved C7 38.5 mm to (160.0, 117.0)
- moved U10 38.2 mm to (156.2, 117.3)
- moved C6 37.2 mm to (157.8, 121.0)
- moved J18 32.5 mm to (228.6, 78.4)
- moved R49 29.1 mm to (188.2, 101.0)
- moved R63 28.9 mm to (191.0, 95.6), turned to 180 degrees
- moved R62 26.9 mm to (191.0, 92.9), turned to 0 degrees
- moved R65 26.4 mm to (190.9, 87.1)
- moved R35 26.3 mm to (191.1, 98.4), turned to 0 degrees
- moved R64 25.9 mm to (191.1, 90.0), turned to 0 degrees
- moved J6 18.5 mm to (228.5, 84.5)
- moved Q11 18.0 mm to (196.2, 92.6), turned to 90 degrees
- moved Q12 16.3 mm to (195.8, 88.0), turned to 90 degrees
- moved Q9 15.9 mm to (196.2, 97.3), turned to 90 degrees
- moved R73 13.8 mm to (222.6, 89.9), turned to 90 degrees
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Connections:
- U2 pad 33: /control/adc_clk -> /DriveAndSens/C_p
- U2 pad 34: /control/adc_dout -> /DriveAndSens/C_n
- U2 pad 38: /control/adc_din -> /DriveAndSens/B_p
- U2 pad 39: /control/~adc_cs -> /DriveAndSens/B_n
- U2 pad 49: (no net) -> /control/adc_clk
- U2 pad 50: /DriveAndSens/B_p -> /control/adc_dout
- U2 pad 51: /DriveAndSens/B_n -> /control/adc_din
- U2 pad 52: (no net) -> /control/~adc_cs
- U2 pad 71: /DriveAndSens/C_p -> (no net)
- U2 pad 72: /DriveAndSens/C_n -> (no net)
Routing:
- net GND: track 487.6 -> 777.8 mm, vias 11 -> 28
- net +3V3: track 434.8 -> 689.0 mm, vias 6 -> 15
- net +1V2: track 118.9 -> 219.3 mm, vias 8 -> 14
- net Net-(R20-Pad1): track 2.82 -> 84.3 mm
- net Net-(Q6-Pad3): track 7.68 -> 73.4 mm
- net Net-(R53-Pad2): track 3.32 -> 68.4 mm
- net /control/adc_clk: track 6.42 -> 71.5 mm
- net /control/adc_dout: track 4.97 -> 70.0 mm
- net +36V: track 201.2 -> 265.7 mm
- net /DriveAndSens/B_p: track 0.00 -> 62.3 mm, vias 0 -> 1
- net /DriveAndSens/B_out: track 34.5 -> 90.2 mm, vias 0 -> 1
- net Net-(R7-Pad2): track 6.20 -> 61.8 mm, vias 0 -> 3
- net +2V5: track 52.2 -> 98.3 mm, vias 1 -> 4
- net Net-(Q10-Pad3): track 9.61 -> 50.0 mm, vias 0 -> 2
- net /control/spare_2: track 54.3 -> 22.5 mm, vias 1 -> 0
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
Commit message: work on  schema
Parts:
- F1: footprint Fuse:Fuse_2512_6332Metric -> my:fuse_20mm
- moved R56 13.2 mm to (182.4, 122.9)
- moved F1 3.25 mm to (218.1, 118.2)
- moved C8 1.59 mm to (214.2, 114.1)
Routing:
- net GND: track 777.8 -> 837.0 mm, vias 28 -> 29
- net +3V3: track 689.0 -> 746.0 mm, vias 15 -> 18
- net Net-(C11-Pad1): track 76.3 -> 127.1 mm, vias 3 -> 2
- net Net-(C17-Pad1): track 56.0 -> 46.3 mm
- net Net-(C10-Pad1): track 38.5 -> 47.2 mm
- net Net-(R56-Pad1): track 14.9 -> 6.66 mm
- net +1V2: track 219.3 -> 216.4 mm
- net Net-(F1-Pad2): track 17.0 -> 19.9 mm, vias 0 -> 1
- net /control/A4: track 31.5 -> 33.5 mm
- net /control/A2: track 24.5 -> 25.7 mm
Other:
- net class Default: trace_width 0.2 -> 0.6
- net class small: trace_width 0.2 -> 0.4

Commit message: work on schema
Parts:
- moved C8 0.50 mm to (214.2, 114.6)
- moved R18 0.27 mm to (143.2, 127.8)
- moved R17 0.19 mm to (138.0, 127.8)
Connections:
- net /control/SI_1 renamed /control/MI_1
- net /control/SO_1 renamed /control/MO_1
Routing:
- net +3V3: track 746.0 -> 747.9 mm
- net (no net): track 0.79 -> 0.00 mm
- net /control/TDI: track 33.1 -> 32.5 mm
- added copper zone on B.Cu, net GND
- added copper zone on F.Cu, net GND
Other:
- net class Default: trace_width 0.6 -> 0.2
- net class small: trace_width 0.4 -> 0.2

Commit message: fix  bug in  schem
Parts:
- U3: moved to B.Cu
- moved R16 18.1 mm to (152.0, 131.4)
- moved R19 11.4 mm to (137.5, 127.7)
- moved U3 10.9 mm to (148.2, 130.7)
- moved R17 10.1 mm to (148.1, 127.7)
- moved T1 2.27 mm to (203.9, 75.6)
- moved T2 0.18 mm to (217.7, 75.8)
- moved T5 0.13 mm to (142.9, 75.5)
- moved R18 0.12 mm to (143.1, 127.7)
- moved T6 0.07 mm to (160.8, 75.6)
Connections:
- T2 pad 2: +36V -> /DriveAndSens/A_out
- T2 pad 3: /DriveAndSens/A_out -> +36V
- T4 pad 2: +36V -> /DriveAndSens/B_out
- T4 pad 3: /DriveAndSens/B_out -> +36V
- T6 pad 2: +36V -> /DriveAndSens/C_out
- T6 pad 3: /DriveAndSens/C_out -> +36V
Routing:
- net /control/TCK: track 24.3 -> 43.9 mm
- net +36V: track 265.7 -> 277.6 mm, vias 1 -> 2
- net /control/TDO: track 23.1 -> 33.8 mm
- net GND: track 837.0 -> 827.6 mm
- net /control/TDI: track 32.5 -> 24.3 mm, vias 2 -> 0
- net +3V3: track 747.9 -> 744.2 mm
- net /DriveAndSens/C_out: track 96.9 -> 99.8 mm
- net /DriveAndSens/B_out: track 90.2 -> 93.0 mm
- net /control/TMS: track 30.9 -> 28.7 mm
- net /DriveAndSens/A_out: track 80.9 -> 82.7 mm
- net Net-(Q3-Pad3): track 77.8 -> 76.3 mm
Other:
- net class energy: trace_width 2.5 -> 2

Commit message: changes in schema
Parts:
- removed Q5, Q8: BC817, Package_TO_SOT_SMD:SOT-23
- removed R22, R59: 20k, Resistor_SMD:R_1206_3216Metric
- added Q14: BC807, Package_TO_SOT_SMD:SOT-23, B.Cu at (212.5, 102.8)
- added Q15: BC807, Package_TO_SOT_SMD:SOT-23, B.Cu at (193.1, 112.0)
- added Q16: BC817, Package_TO_SOT_SMD:SOT-23, B.Cu at (192.3, 107.9)
- added Q17: BC807, Package_TO_SOT_SMD:SOT-23, B.Cu at (160.3, 113.6)
- added Q18: BC817, Package_TO_SOT_SMD:SOT-23, B.Cu at (154.5, 115.1)
- added R27: 20k, Resistor_SMD:R_1206_3216Metric, B.Cu at (188.2, 110.9)
- added R3: 20k, Resistor_SMD:R_1206_3216Metric, B.Cu at (188.1, 108.2)
- added R6: 20k, Resistor_SMD:R_1206_3216Metric, B.Cu at (193.4, 115.2)
- added R75: 20k, Resistor_SMD:R_1206_3216Metric, B.Cu at (188.1, 113.8)
- added R76: 20k, Resistor_SMD:R_1206_3216Metric, B.Cu at (207.3, 103.6)
- added R77: 20k, Resistor_SMD:R_1206_3216Metric, B.Cu at (166.6, 109.9)
- added R78: 20k, Resistor_SMD:R_1206_3216Metric, B.Cu at (151.2, 115.2)
- added R79: 20k, Resistor_SMD:R_1206_3216Metric, B.Cu at (158.6, 109.4)
- added R80: 20k, Resistor_SMD:R_1206_3216Metric, B.Cu at (164.1, 106.4)
- added R81: 20k, Resistor_SMD:R_1206_3216Metric, B.Cu at (158.6, 117.0)
- added R82: 20k, Resistor_SMD:R_1206_3216Metric, B.Cu at (153.0, 110.7)
- added R83: 10k, Resistor_SMD:R_1206_3216Metric, F.Cu at (160.1, 129.3)
- added R84: 10k, Resistor_SMD:R_1206_3216Metric, F.Cu at (162.8, 129.3)
- added R85: 10k, Resistor_SMD:R_1206_3216Metric, F.Cu at (165.7, 129.3)
- D11: value hal_err -> done
- R1, R2, R23, R26, R34, R4: value 50k -> 20k
- R20: value 2.4 -> 4.8k
- R5, R53, R7: value 1k -> 2k
- R58, R8: value 2.4k -> 4.8k
- R67, R73: value 4.7k -> 640
- moved R34 49.1 mm to (201.5, 104.9), turned to 270 degrees
- moved R26 38.8 mm to (197.2, 109.2), turned to 0 degrees
- moved R4 20.3 mm to (212.4, 111.6)
- moved R71 16.6 mm to (113.0, 94.1), turned to 180 degrees
- moved R23 7.82 mm to (205.5, 109.8)
- moved R72 7.16 mm to (113.0, 90.7), turned to 0 degrees
- moved R70 6.94 mm to (108.5, 84.1), turned to 270 degrees
- moved R21 6.92 mm to (217.4, 106.9), turned to 90 degrees
- moved R24 6.72 mm to (185.8, 105.3)
- moved Q2 6.09 mm to (197.4, 103.2)
- moved R69 5.77 mm to (105.5, 84.2)
- moved R1 3.74 mm to (213.4, 105.9), turned to 0 degrees
- moved Q6 3.35 mm to (183.8, 108.6)
- moved J15 2.79 mm to (228.3, 104.9)
- moved Q7 2.71 mm to (161.8, 109.5)
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Connections:
- J13 pad 3: /control/hal_C -> Net-(J13-Pad3)
- J13 pad 4: /control/hal_B -> Net-(J13-Pad4)
- J13 pad 5: /control/hal_A -> Net-(J13-Pad5)
- Q4 pad 2: GND -> Net-(Q4-Pad2)
- Q4 pad 3: Net-(Q3-Pad1) -> +3V3
- R1 pad 2: Net-(Q1-Pad1) -> Net-(Q14-Pad1)
- R2 pad 2: Net-(Q2-Pad1) -> Net-(Q15-Pad1)
- R21 pad 1: +36V -> Net-(Q14-Pad3)
- R21 pad 2: Net-(Q3-Pad1) -> Net-(Q1-Pad1)
- R26 pad 1: /DriveAndSens/C_p -> Net-(Q15-Pad3)
- R26 pad 2: Net-(Q7-Pad1) -> Net-(Q2-Pad1)
- R34 pad 1: /DriveAndSens/C_n -> Net-(Q4-Pad2)
- R34 pad 2: Net-(Q8-Pad1) -> GND
- R4 pad 1: /DriveAndSens/B_n -> Net-(Q14-Pad3)
- R4 pad 2: Net-(Q5-Pad1) -> GND
Routing:
- net +3V3: track 744.2 -> 835.3 mm, vias 18 -> 21
- net +36V: track 277.6 -> 297.4 mm
- net /control/A1: track 38.7 -> 25.3 mm
- net Net-(Q14-Pad3): track 0.00 -> 13.0 mm
- net Net-(Q17-Pad3): track 0.00 -> 11.0 mm
- net GND: track 827.6 -> 838.5 mm, vias 29 -> 31
- net Net-(Q15-Pad1): track 0.00 -> 9.45 mm
- net Net-(Q18-Pad2): track 0.00 -> 8.59 mm
- net Net-(Q17-Pad1): track 0.00 -> 8.06 mm
- net Net-(Q3-Pad3): track 76.3 -> 83.4 mm
- net Net-(Q15-Pad3): track 0.00 -> 6.91 mm
- net Net-(Q4-Pad2): track 0.00 -> 6.70 mm
- net /control/A4: track 33.5 -> 27.0 mm
- net /DriveAndSens/C_p: track 37.6 -> 43.9 mm
- net Net-(Q16-Pad2): track 0.00 -> 6.05 mm
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